File: kicad/blossom.kicad_pcb (KiCad board)
At the start: 2 copper layers, 48.7 x 48.7 mm, 38 parts, among them J1 AVR-ISP-6, SW1 SW_Push, SW2 SW_Push, SW3 SW_Push, U1 ATtiny85-10SU

Commit message: Migrate to KiCad 6
Parts:
- U1: value ATtiny85-10SU -> ATtiny85V-10SU; footprint Package_SO:SOIJ-8_5.3x5.3mm_P1.27mm -> Package_SO:SOIC-8W_5.3x5.3mm_P1.27mm
- moved J1 11.6 mm to (148.6, 78.8), turned to -135 degrees
- moved BT1 0.71 mm to (139.7, 89.4)
Routing:
- net PB2: track 20.5 -> 12.1 mm
- net PB0: track 17.6 -> 23.6 mm, vias 0 -> 4
- net +3V3: track 62.5 -> 67.1 mm, vias 4 -> 3
- net PB1: track 19.9 -> 15.5 mm, vias 0 -> 2
- net Net-(D1-Pad2): track 108.0 -> 104.2 mm
- net PB5: track 19.4 -> 15.8 mm
- net GND: track 12.8 -> 10.3 mm, vias 3 -> 4
- net Net-(D10-Pad1): track 106.7 -> 104.3 mm, vias 3 -> 4
- net C2: track 4.74 -> 4.01 mm
- net Net-(R7-Pad2): track 23.8 -> 23.2 mm
Other:
- net class Default removed
